File: KiCad/Etherscape.kicad_sch (KiCad schematic)
At the start: 27 parts, among them J1 AudioJack3, J2 USB_C_Receptacle, J4 Conn_01x01_Female, J6 Conn_01x01_Female, J8 Raspberry_Pi_2_3, U1 DW01, U2 TP4056, U3 FS8205A

Commit message: added KiCad files
Parts:
- added R11, R12: 1.8K, symbol Device:R
- added U4: 74HC595, Package_SO:SOIC-16W_5.3x10.2mm_P1.27mm, symbol 74xx:74HC595
Connections:
- net Earth: now also J1.R, J1.S, R11.1, R12.2
- net at C7.1: now also J1.T, R12.1
- net AUDIO_LED: now reaches J8.29 (GCLK1/GPIO5)
- net at C6.1: now also R11.2
Other:
- moved on the sheet: C4, C5, C6, C7, J1, R10, R7, R8, R9

Commit message: updated schematic
Parts:
- added D3, D4, D5, D6, D7, D8, D9: LED, LED_SMD:LED_1206_3216Metric, symbol Device:LED
- added R13, R14, R15, R18: 50, Resistor_SMD:R_0603_1608Metric, symbol Device:R
- added R16: 75, Resistor_SMD:R_0603_1608Metric, symbol Device:R
- added R17, R19: 80, Resistor_SMD:R_0603_1608Metric, symbol Device:R
- added R20, R21, R22, R23: 10K, Resistor_SMD:R_0603_1608Metric, symbol Device:R
- added SW1, SW2, SW3, SW4: SW_Push, symbol Switch:SW_Push
- added SW5: SW_DIP_x01, symbol Switch:SW_DIP_x01
Connections:
- net Earth: now also U4.13 (~{OE}), U4.8 (GND), R20.2, R21.2, R22.2, R23.2
- net VIN: now also SW5.1; no longer C3.1, D1.2 (A), D2.2 (A), U2.4 (VCC), U2.8 (CE), U2.9 (PP)
- net at U4.1 (QB): now also R13.1
- net 74HC595_SRCLK: now reaches U4.11 (SRCLK)
- net 74HC595_SRCLK: now also J8.38 (GPIO20/MOSI1)
- net 74HC595_RCLK: now reaches U4.12 (RCLK)
- net 74HC595_RCLK: now also J8.40 (GPIO21/SCLK1)
- net 74HC595_SER: now reaches U4.14 (SER)
- net 74HC595_SER: now also J8.36 (GPIO16)
- net 74HC595_VCC: now reaches U4.16 (VCC)
- net at U4.2 (QC): now also R14.1
- net at U4.3 (QD): now also R15.1
- net at U4.4 (QE): now also R16.1
- net at U4.5 (QF): now also R17.1
- net at U4.6 (QG): now also R18.1
- net at U4.7 (QH): now also R19.1
- net +3V3: now reaches J8.1 (3V3)
- net +3V3: now also SW1.1, SW2.1, SW3.1, SW4.1
- net VOL_UP_BUTTON: now reaches J8.13 (GPIO27)
- net VOL_UP_BUTTON: now also R22.1, SW3.2
- net REC_BUTTON: now reaches J8.15 (GPIO22)
- net REC_BUTTON: now also R21.1, SW2.2
- net BAT_BUTTON: now reaches J8.16 (GPIO23)
- net BAT_BUTTON: now also R20.1, SW1.2
- net VOL_DOWN_BUTTON: now reaches J8.37 (GPIO26)
- net VOL_DOWN_BUTTON: now also R23.1, SW4.2
- new net: C3.1, D1.2 (A), D2.2 (A), SW5.2, U2.4 (VCC), U2.8 (CE), U2.9 (PP)
- new net: D7.2 (A), R17.2
- new net: D6.2 (A), R16.2
- new net: D9.2 (A), R19.2
- new net: D5.2 (A), R15.2
- new net: D4.2 (A), R14.2
- new net: D3.2 (A), R13.2
- new net: D8.2 (A), R18.2
- no-connect marks 20 -> 21
Other:
- note added: "Control Knobs (Volume, Record, On/Off, Battery Status)"
- note added: "On/Off"
- note added: "Raspberry Pi Zero W GPIO"
- note added: "Record"
- note added: "VU Meter/Battery Indicator"
- note removed: "Control Knobs (Volume, Record, On/Off)"
- moved on the sheet: C1, C2, C3, C4, C5, C6, C7, D1, D2, J1, J2, J4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
